Commit message: Add some mounts to head urdf
Add coarse meshes
Position mic mount and camera mount with consistent dimensions
Add launch file for quickly visualizing the URDF (without going through gazebo)

File: astro_description/urdf/head.xacro (robot description, xacro)
@@ -1,4 +1,5 @@
 <?xml version="1.0"?>
 <robot xmlns:xacro="http://www.ros.org/wiki/xacro" name="head">
+    <xacro:include filename="$(find realsense2_description)/urdf/_d415.urdf.xacro"/>
     <xacro:macro name="head">
         <link name="head_pan_link">
@@ -165,5 +166,5 @@
             <child link="head_camera_depth_optical_frame" />
         </joint>
-        <link name="head_external_camera_link">
+        <link name="head_external_camera_mount_link">
             <inertial>
                 <origin rpy="0 0 0" xyz="0.00 -0.0025 0.013" />
@@ -174,8 +175,8 @@
                 <origin rpy="0 0 0" xyz="0 0 0" />
                 <geometry>
-                       <box size="0.020 0.099 0.023" />
-                </geometry>
-                <material name="">
-                    <color rgba="0.086 0.506 0.767 1" />
+                       <mesh filename="package://astro_description/meshes/head_external_camera_mount_link.stl" />
+                </geometry>
+                <material name="">
+                    <color rgba="0.20 0.20 0.20 1" />
                 </material>
             </visual>
@@ -188,11 +189,14 @@
         </link>
         <joint name="head_external_camera_joint" type="fixed">
-            <origin rpy="0 0 0" xyz="0.03 0.05 0.067" />
+            <origin rpy="0 0 0" xyz="0.01 0.0625 0.055" />
             <parent link="head_tilt_link" />
-            <child link="head_external_camera_link" />
-        </joint>
-        <link name="head_mic_link">
-            <inertial>
-                <origin rpy="0 0 0" xyz="0.00 -0.0025 0.013" />
+            <child link="head_external_camera_mount_link" />
+        </joint>
+        <sensor_r435 name="Head Camera" parent="head_external_camera_mount_joint">
+            <origin xyz="0 0 0" rpy="1 0 0"/>
+        </sensor_r435>
+        <link name="head_mic_mount_link">
+            <inertial>
+                <origin rpy="0 0 0" xyz="0.00 0.00 0.00" />
                 <mass value="0.072" />
                 <inertia ixx="0.0061" ixy="-0.0" ixz="0.0002" iyy="0.0014" iyz="-0.0001" izz="0.0061" />
@@ -201,8 +205,8 @@
                 <origin rpy="0 0 0" xyz="0 0 0" />
                 <geometry>
-                       <cylinder radius="0.035" length="0.003" />
-                </geometry>
-                <material name="">
-                    <color rgba="0.086 0.506 0.767 1" />
+                       <mesh filename="package://astro_description/meshes/mic_mount_link.stl" />
+                </geometry>
+                <material name="">
+                    <color rgba="0.20 0.20 0.20 1" />
                 </material>
             </visual>
@@ -215,7 +219,7 @@
         </link>
         <joint name="head_mic_joint" type="fixed">
-            <origin rpy="0 0 0" xyz="0.017 -0.055 0.06" />
+            <origin rpy="0 0 0" xyz="0.035 -0.0625 0.055" />
             <parent link="head_tilt_link" />
-            <child link="head_mic_link" />
+            <child link="head_mic_mount_link" />
         </joint>
     </xacro:macro>

Commit message: Add display and xavier to head URDF
Fix up visuals

File: astro_description/urdf/head.xacro (robot description, xacro)
@@ -42,7 +42,7 @@
             </actuator>
         </transmission>
-        <link name="head_computer_link">
-            <inertial>
-                <origin rpy="0 0 0" xyz="0.0321 0.0161 0.0390" />
+        <link name="xavier_mount">
+            <inertial>
+                <origin rpy="0 0 0" xyz="0 0 0" />
                 <!-- Estimate -->
                 <mass value="0.5" />
@@ -52,8 +52,36 @@
                 <origin rpy="0 0 0" xyz="0 0 0" />
                 <geometry>
+                    <mesh filename="package://astro_description/meshes/xavier_mount.stl" />
+                </geometry>
+                <material name="">
+                    <color rgba="0.2 0.2 0.2 1" />
+                </material>
+            </visual>
+            <collision>
+                <origin rpy="0 0 0" xyz="0 0 0" />
+                <geometry>
                     <box size="0.105 0.105 0.066"/>
                 </geometry>
-                <material name="">
-                    <color rgba="1.0 1.0 1.0 1" />
+            </collision>
+        </link>
+        <joint name="xavier_mount_joint" type="fixed">
+            <origin rpy="0.0 0.0 0.0" xyz="0.05 0.0625 0.09" />
+            <parent link="head_pan_link" />
+            <child link="xavier_mount" />
+        </joint>
+        <link name="xavier">
+            <inertial>
+                <origin rpy="0 0 0" xyz="0 0 0" />
+                <!-- Estimate -->
+                <mass value="0.5" />
+                <inertia ixx="0.0129" ixy="0.0002" ixz="0.0007" iyy="0.0095" iyz="-0.0" izz="0.0184" />
+            </inertial>
+            <visual>
+                <origin rpy="0 0 0" xyz="0 0 0" />
+                <geometry>
+                    <mesh filename="package://astro_description/meshes/xavier.stl" />
+                </geometry>
+                <material name="">
+                    <color rgba="0.3 0.3 0.3 1" />
                 </material>
             </visual>
@@ -65,12 +93,40 @@
             </collision>
         </link>
-        <joint name="head_computer_link" type="fixed">
-            <origin rpy="0.0 0.0 0.0" xyz="-0.05 0 0.13" />
+        <joint name="xavier_joint" type="fixed">
+            <origin rpy="0.0 0.0 0.0" xyz="-0.109 -0.104 0.0265" />
+            <parent link="xavier_mount" />
+            <child link="xavier" />
+        </joint>
+        <link name="head_display_mount">
+            <inertial>
+                <origin rpy="0 0 0" xyz="0 0 0" />
+                <!-- Estimate -->
+                <mass value="0.5" />
+                <inertia ixx="0.0129" ixy="0.0002" ixz="0.0007" iyy="0.0095" iyz="-0.0" izz="0.0184" />
+            </inertial>
+            <visual>
+                <origin rpy="0 0 0" xyz="0 0 0" />
+                <geometry>
+                    <mesh filename="package://astro_description/meshes/display_mount.stl" />
+                </geometry>
+                <material name="">
+                    <color rgba="0.2 0.2 0.2 1" />
+                </material>
+            </visual>
+            <collision>
+                <origin rpy="0 0 0" xyz="0 0 0" />
+                <geometry>
+                    <box size="0.105 0.105 0.066"/>
+                </geometry>
+            </collision>
+        </link>
+        <joint name="head_display_mount_joint" type="fixed">
+            <origin rpy="0.0 0.0 0.0" xyz="0.075 0.0625 0.09" />
             <parent link="head_pan_link" />
-            <child link="head_computer_link" />
-        </joint>
-       <link name="head_display_link">
-            <inertial>
-                <origin rpy="0 0 0" xyz="0.0321 0.0161 0.0390" />
+            <child link="head_display_mount" />
+        </joint>
+       <link name="head_display">
+            <inertial>
+                <origin rpy="0 0 0" xyz="0 0 0" />
                 <mass value="1.0" />
                 <inertia ixx="0.0129" ixy="0.0002" ixz="0.0007" iyy="0.0095" iyz="-0.0" izz="0.0184" />
@@ -79,8 +135,8 @@
                 <origin rpy="0 0 0" xyz="0 0 0" />
                 <geometry>
-                    <box size="0.02 0.23 0.1524"/>
-                </geometry>
-                <material name="">
-                    <color rgba="1.0 1.0 1.0 1" />
+                    <mesh filename="package://astro_description/meshes/head_display.stl" />
+                </geometry>
+                <material name="">
+                    <color rgba="0.2 0.2 0.2 1" />
                 </material>
             </visual>
@@ -92,8 +148,8 @@
             </collision>
         </link>
-        <joint name="head_display_link_joint" type="fixed">
-            <origin rpy="0.0 -0.6 0.0" xyz="0.05 0 0.19" />
-            <parent link="head_pan_link" />
-            <child link="head_display_link" />
+        <joint name="head_display_joint" type="fixed">
+            <origin rpy="1.0472 0.0 1.56" xyz="-0.05 -0.063 0.095" />
+            <parent link="head_display_mount" />
+            <child link="head_display" />
         </joint>
         <link name="head_tilt_link">
@@ -166,5 +222,5 @@
             <child link="head_camera_depth_optical_frame" />
         </joint>
-        <link name="head_external_camera_mount_link">
+        <link name="head_external_camera_mount">
             <inertial>
                 <origin rpy="0 0 0" xyz="0.00 -0.0025 0.013" />
@@ -175,5 +231,5 @@
                 <origin rpy="0 0 0" xyz="0 0 0" />
                 <geometry>
-                       <mesh filename="package://astro_description/meshes/head_external_camera_mount_link.stl" />
+                       <mesh filename="package://astro_description/meshes/head_external_camera_mount.stl" />
                 </geometry>
                 <material name="">
@@ -188,13 +244,14 @@
             </collision>
         </link>
-        <joint name="head_external_camera_joint" type="fixed">
+        <joint name="head_external_camera_mount_joint" type="fixed">
             <origin rpy="0 0 0" xyz="0.01 0.0625 0.055" />
             <parent link="head_tilt_link" />
-            <child link="head_external_camera_mount_link" />
-        </joint>
-        <sensor_r435 name="Head Camera" parent="head_external_camera_mount_joint">
-            <origin xyz="0 0 0" rpy="1 0 0"/>
-        </sensor_r435>
-        <link name="head_mic_mount_link">
+            <child link="head_external_camera_mount" />
+        </joint>
+        <xacro:arg name="use_nominal_extrinsics" default="True" />
+        <sensor_d415 name="head_external_camera" parent="head_external_camera_mount" use_nominal_extrinsics="true">
+            <origin xyz="0.025 -0.025 0.003" rpy="0 0 0"/>
+        </sensor_d415>
+        <link name="head_mic_mount">
             <inertial>
                 <origin rpy="0 0 0" xyz="0.00 0.00 0.00" />
@@ -205,5 +262,5 @@
                 <origin rpy="0 0 0" xyz="0 0 0" />
                 <geometry>
-                       <mesh filename="package://astro_description/meshes/mic_mount_link.stl" />
+                       <mesh filename="package://astro_description/meshes/mic_mount.stl" />
                 </geometry>
                 <material name="">
@@ -218,8 +275,62 @@
             </collision>
         </link>
-        <joint name="head_mic_joint" type="fixed">
+        <joint name="head_mic_mount_joint" type="fixed">
             <origin rpy="0 0 0" xyz="0.035 -0.0625 0.055" />
             <parent link="head_tilt_link" />
-            <child link="head_mic_mount_link" />
+            <child link="head_mic_mount" />
+        </joint>
+        <link name="head_mic">
+            <inertial>
+                <origin rpy="0 0 0" xyz="0.00 0.00 0.00" />
+                <mass value="0.072" />
+                <inertia ixx="0.0061" ixy="-0.0" ixz="0.0002" iyy="0.0014" iyz="-0.0001" izz="0.0061" />
+            </inertial>
+            <visual>
+                <origin rpy="0 0 0" xyz="0 0 0" />
+                <geometry>
+                       <mesh filename="package://astro_description/meshes/mic.stl" />
+                </geometry>
+                <material name="">
+                    <color rgba="0.20 0.20 0.20 1" />
+                </material>
+            </visual>
+            <collision>
+                <origin rpy="0 0 0" xyz="0 0 0" />
+                <geometry>
+                    <box size="0.07 0.07 0.003" />
+                </geometry>
+            </collision>
+        </link>
+        <joint name="head_mic_joint" type="fixed">
+            <origin rpy="0 0 -1.56" xyz="-0.013 0.007 0.022" />
+            <parent link="head_mic_mount" />
+            <child link="head_mic" />
+        </joint>
+                <link name="mic_shell">
+            <inertial>
+                <origin rpy="0 0 0" xyz="0.00 0.00 0.00" />
+                <mass value="0.072" />
+                <inertia ixx="0.0061" ixy="-0.0" ixz="0.0002" iyy="0.0014" iyz="-0.0001" izz="0.0061" />
+            </inertial>
+            <visual>
+                <origin rpy="0 0 0" xyz="0 0 0" />
+                <geometry>
+                       <mesh filename="package://astro_description/meshes/mic_shell.stl" />
+                </geometry>
+                <material name="">
+                    <color rgba="0.90 0.88 0.81 1" />
+                </material>
+            </visual>
+            <collision>
+                <origin rpy="0 0 0" xyz="0 0 0" />
+                <geometry>
+                    <box size="0.07 0.07 0.003" />
+                </geometry>
+            </collision>
+        </link>
+        <joint name="mic_shell_joint" type="fixed">
+            <origin rpy="0 0 0" xyz="0.0 0.0 0.0" />
+            <parent link="head_mic_mount" />
+            <child link="mic_shell" />
         </joint>
     </xacro:macro>
