Commit message: Fix head URDF collisions and inertia properties
Tilt unit works in simulation again

File: astro_description/urdf/head.xacro (robot description, xacro)
@@ -5,30 +5,30 @@
         <link name="head_pan_link">
             <inertial>
-                <origin rpy="0 0 0" xyz="0.0321 0.0161 0.0390" />
-                <mass value="2.2556" />
-                <inertia ixx="0.0129" ixy="0.0002" ixz="0.0007" iyy="0.0095" iyz="-0.0" izz="0.0184" />
-            </inertial>
-            <visual>
-                <origin rpy="0 0 0" xyz="0 0 0" />
-                <geometry>
-                    <mesh filename="package://fetch_description/meshes/head_pan_link.dae" />
-                </geometry>
-                <material name="">
-                    <color rgba="0.356 0.361 0.376 1" />
-                </material>
-            </visual>
-            <collision>
-                <origin rpy="0 0 0" xyz="0 0 0" />
-                <geometry>
-                    <mesh filename="package://fetch_description/meshes/head_pan_link_collision.STL" />
+                <origin rpy="0 0 0" xyz="0.0321 0.0161 0.0390"/>
+                <mass value="2.2556"/>
+                <inertia ixx="0.0129" ixy="0.0002" ixz="0.0007" iyy="0.0095" iyz="-0.0" izz="0.0184"/>
+            </inertial>
+            <visual>
+                <origin rpy="0 0 0" xyz="0 0 0"/>
+                <geometry>
+                    <mesh filename="package://fetch_description/meshes/head_pan_link.dae"/>
+                </geometry>
+                <material name="">
+                    <color rgba="0.356 0.361 0.376 1"/>
+                </material>
+            </visual>
+            <collision>
+                <origin rpy="0 0 0" xyz="0 0 0"/>
+                <geometry>
+                    <mesh filename="package://fetch_description/meshes/head_pan_link_collision.STL"/>
                 </geometry>
             </collision>
         </link>
         <joint name="head_pan_joint" type="revolute">
-            <origin rpy="0 0 0" xyz="0.053125 0 0.603001417713939" />
-            <parent link="torso_lift_link" />
-            <child link="head_pan_link" />
-            <axis xyz="0 0 1" />
-            <limit effort="0.32" lower="-1.57" upper="1.57" velocity="1.57" />
+            <origin rpy="0 0 0" xyz="0.053125 0 0.603001417713939"/>
+            <parent link="torso_lift_link"/>
+            <child link="head_pan_link"/>
+            <axis xyz="0 0 1"/>
+            <limit effort="0.32" lower="-1.57" upper="1.57" velocity="1.57"/>
         </joint>
         <transmission name="head_pan_joint_tran">
@@ -44,20 +44,48 @@
         <link name="xavier_mount">
             <inertial>
-                <origin rpy="0 0 0" xyz="0 0 0" />
+                <origin rpy="0 0 0" xyz="0 0 0"/>
                 <!-- Estimate -->
-                <mass value="0.5" />
-                <inertia ixx="0.0129" ixy="0.0002" ixz="0.0007" iyy="0.0095" iyz="-0.0" izz="0.0184" />
-            </inertial>
-            <visual>
-                <origin rpy="0 0 0" xyz="0 0 0" />
-                <geometry>
-                    <mesh filename="package://astro_description/meshes/xavier_mount.stl" />
-                </geometry>
-                <material name="">
-                    <color rgba="0.2 0.2 0.2 1" />
-                </material>
-            </visual>
-            <collision>
-                <origin rpy="0 0 0" xyz="0 0 0" />
+                <mass value="0.25"/>
+                <inertia ixx="0.0129" ixy="0.0002" ixz="0.0007" iyy="0.0095" iyz="-0.0" izz="0.0184"/>
+            </inertial>
+            <visual>
+                <origin rpy="0 0 0" xyz="0 0 0"/>
+                <geometry>
+                    <mesh filename="package://astro_description/meshes/xavier_mount.stl"/>
+                </geometry>
+                <material name="">
+                    <color rgba="0.2 0.2 0.2 1"/>
+                </material>
+            </visual>
+            <collision>
+                <origin rpy="0 0 0" xyz="-0.05 -0.0625 0.01"/>
+                <geometry>
+                    <box size="0.125 0.105 0.03"/>
+                </geometry>
+            </collision>
+        </link>
+        <joint name="xavier_mount_joint" type="fixed">
+            <origin rpy="0.0 0.0 0.0" xyz="0.05 0.0625 0.09"/>
+            <parent link="head_pan_link"/>
+            <child link="xavier_mount"/>
+        </joint>
+        <link name="xavier">
+            <inertial>
+                <origin rpy="0 0 0" xyz="0 0 0"/>
+                <!-- Estimate -->
+                <mass value="0.5"/>
+                <inertia ixx="0.0129" ixy="0.0002" ixz="0.0007" iyy="0.0095" iyz="-0.0" izz="0.0184"/>
+            </inertial>
+            <visual>
+                <origin rpy="0 0 0" xyz="0 0 0"/>
+                <geometry>
+                    <mesh filename="package://astro_description/meshes/xavier.stl"/>
+                </geometry>
+                <material name="">
+                    <color rgba="0.3 0.3 0.3 1"/>
+                </material>
+            </visual>
+            <collision>
+                <origin rpy="0 0 0" xyz="0.05 0.05 0.0265"/>
                 <geometry>
                     <box size="0.105 0.105 0.066"/>
@@ -65,120 +93,92 @@
             </collision>
         </link>
-        <joint name="xavier_mount_joint" type="fixed">
-            <origin rpy="0.0 0.0 0.0" xyz="0.05 0.0625 0.09" />
-            <parent link="head_pan_link" />
-            <child link="xavier_mount" />
-        </joint>
-        <link name="xavier">
-            <inertial>
-                <origin rpy="0 0 0" xyz="0 0 0" />
+        <joint name="xavier_joint" type="fixed">
+            <origin rpy="0.0 0.0 0.0" xyz="-0.109 -0.104 0.0265"/>
+            <parent link="xavier_mount"/>
+            <child link="xavier"/>
+        </joint>
+        <link name="head_display_mount">
+            <inertial>
+                <origin rpy="0 0 0" xyz="0 0 0"/>
                 <!-- Estimate -->
-                <mass value="0.5" />
-                <inertia ixx="0.0129" ixy="0.0002" ixz="0.0007" iyy="0.0095" iyz="-0.0" izz="0.0184" />
-            </inertial>
-            <visual>
-                <origin rpy="0 0 0" xyz="0 0 0" />
-                <geometry>
-                    <mesh filename="package://astro_description/meshes/xavier.stl" />
-                </geometry>
-                <material name="">
-                    <color rgba="0.3 0.3 0.3 1" />
-                </material>
-            </visual>
-            <collision>
-                <origin rpy="0 0 0" xyz="0 0 0" />
-                <geometry>
-                    <box size="0.105 0.105 0.066"/>
-                </geometry>
-            </collision>
-        </link>
-        <joint name="xavier_joint" type="fixed">
-            <origin rpy="0.0 0.0 0.0" xyz="-0.109 -0.104 0.0265" />
-            <parent link="xavier_mount" />
-            <child link="xavier" />
-        </joint>
-        <link name="head_display_mount">
-            <inertial>
-                <origin rpy="0 0 0" xyz="0 0 0" />
-                <!-- Estimate -->
-                <mass value="0.5" />
-                <inertia ixx="0.0129" ixy="0.0002" ixz="0.0007" iyy="0.0095" iyz="-0.0" izz="0.0184" />
-            </inertial>
-            <visual>
-                <origin rpy="0 0 0" xyz="0 0 0" />
-                <geometry>
-                    <mesh filename="package://astro_description/meshes/display_mount.stl" />
-                </geometry>
-                <material name="">
-                    <color rgba="0.2 0.2 0.2 1" />
-                </material>
-            </visual>
-            <collision>
-                <origin rpy="0 0 0" xyz="0 0 0" />
-                <geometry>
-                    <box size="0.105 0.105 0.066"/>
+                <mass value="0.25"/>
+                <inertia ixx="0.0129" ixy="0.0002" ixz="0.0007" iyy="0.0095" iyz="-0.0" izz="0.0184"/>
+            </inertial>
+            <visual>
+                <origin rpy="0 0 0" xyz="0 0 0"/>
+                <geometry>
+                    <mesh filename="package://astro_description/meshes/display_mount.stl"/>
+                </geometry>
+                <material name="">
+                    <color rgba="0.2 0.2 0.16 1"/>
+                </material>
+            </visual>
+            <collision>
+                <origin rpy="0 0 0" xyz="-.08 -.08 .09"/>
+                <geometry>
+                    <box size="0.105 0.105 0.18"/>
                 </geometry>
             </collision>
         </link>
         <joint name="head_display_mount_joint" type="fixed">
-            <origin rpy="0.0 0.0 0.0" xyz="0.075 0.0625 0.09" />
-            <parent link="head_pan_link" />
-            <child link="head_display_mount" />
-        </joint>
-       <link name="head_display">
-            <inertial>
-                <origin rpy="0 0 0" xyz="0 0 0" />
-                <mass value="1.0" />
-                <inertia ixx="0.0129" ixy="0.0002" ixz="0.0007" iyy="0.0095" iyz="-0.0" izz="0.0184" />
-            </inertial>
-            <visual>
-                <origin rpy="0 0 0" xyz="0 0 0" />
-                <geometry>
-                    <mesh filename="package://astro_description/meshes/head_display.stl" />
-                </geometry>
-                <material name="">
-                    <color rgba="0.2 0.2 0.2 1" />
-                </material>
-            </visual>
-            <collision>
-                <origin rpy="0 0 0" xyz="0 0 0" />
-                <geometry>
-                    <box size="0.1524 0.23 0.02"/>
+            <origin rpy="0.0 0.0 0.0" xyz="0.075 0.0625 0.09"/>
+            <parent link="head_pan_link"/>
+            <child link="head_display_mount"/>
+        </joint>
+        <link name="head_display">
+            <inertial>
+                <origin rpy="0 0 0" xyz="0 0 0"/>
+                <mass value="1.0"/>
+                <inertia ixx="0.0129" ixy="0.0002" ixz="0.0007" iyy="0.0095" iyz="-0.0" izz="0.0184"/>
+            </inertial>
+            <visual>
+                <origin rpy="0 0 0" xyz="0 0 0"/>
+                <geometry>
+                    <mesh filename="package://astro_description/meshes/head_display.stl"/>
+                </geometry>
+                <material name="">
+                    <color rgba="0.2 0.2 0.2 1"/>
+                </material>
+            </visual>
+            <collision>
+                <origin rpy="0 0 0" xyz="0 0 0"/>
+                <geometry>
+                    <box size="0.23 0.1524  0.02"/>
                 </geometry>
             </collision>
         </link>
         <joint name="head_display_joint" type="fixed">
-            <origin rpy="1.0472 0.0 1.56" xyz="-0.05 -0.063 0.095" />
-            <parent link="head_display_mount" />
-            <child link="head_display" />
+            <origin rpy="1.0472 0.0 1.56" xyz="-0.05 -0.063 0.095"/>
+            <parent link="head_display_mount"/>
+            <child link="head_display"/>
         </joint>
         <link name="head_tilt_link">
             <inertial>
-                <origin rpy="0 0 0" xyz="0.0081 0.0025 0.0113" />
-                <mass value="0.9087" />
-                <inertia ixx="0.0061" ixy="-0.0" ixz="0.0002" iyy="0.0014" iyz="-0.0001" izz="0.0061" />
-            </inertial>
-            <visual>
-                <origin rpy="0 0 0" xyz="0 0 0" />
-                <geometry>
-                    <mesh filename="package://fetch_description/meshes/head_tilt_link.dae" />
-                </geometry>
-                <material name="">
-                    <color rgba="0.086 0.506 0.767 1" />
-                </material>
-            </visual>
-            <collision>
-                <origin rpy="0 0 0" xyz="0 0 0" />
-                <geometry>
-                    <mesh filename="package://fetch_description/meshes/head_tilt_link_collision.STL" />
+                <origin rpy="0 0 0" xyz="0.0081 0.0025 0.0113"/>
+                <mass value="0.9087"/>
+                <inertia ixx="0.0061" ixy="-0.0" ixz="0.0002" iyy="0.0014" iyz="-0.0001" izz="0.0061"/>
+            </inertial>
+            <visual>
+                <origin rpy="0 0 0" xyz="0 0 0"/>
+                <geometry>
+                    <mesh filename="package://fetch_description/meshes/head_tilt_link.dae"/>
+                </geometry>
+                <material name="">
+                    <color rgba="0.086 0.506 0.767 1"/>
+                </material>
+            </visual>
+            <collision>
+                <origin rpy="0 0 0" xyz="0 0 0"/>
+                <geometry>
+                    <mesh filename="package://fetch_description/meshes/head_tilt_link_collision.STL"/>
                 </geometry>
             </collision>
         </link>
         <joint name="head_tilt_joint" type="revolute">
-            <origin rpy="0 0 0" xyz="0.14253 0 0.057999" />
-            <parent link="head_pan_link" />
-            <child link="head_tilt_link" />
-            <axis xyz="0 1 0" />
-            <limit effort="0.68" lower="-0.76" upper="1.45" velocity="1.57" />
+            <origin rpy="0 0 0" xyz="0.14253 0 0.057999"/>
+            <parent link="head_pan_link"/>
+            <child link="head_tilt_link"/>
+            <axis xyz="0 1 0"/>
+            <limit effort="0.68" lower="-0.76" upper="1.45" velocity="1.57"/>
         </joint>
         <transmission name="head_tilt_joint_tran">
@@ -192,62 +192,62 @@
             </actuator>
         </transmission>
-        <link name="head_camera_link" />
+        <link name="head_camera_link"/>
         <joint name="head_camera_joint" type="fixed">
-            <origin rpy="0 0 0" xyz="0.055 0 0.0225" />
-            <parent link="head_tilt_link" />
-            <child link="head_camera_link" />
-        </joint>
-        <link name="head_camera_rgb_frame" />
+            <origin rpy="0 0 0" xyz="0.055 0 0.0225"/>
+            <parent link="head_tilt_link"/>
+            <child link="head_camera_link"/>
+        </joint>
+        <link name="head_camera_rgb_frame"/>
         <joint name="head_camera_rgb_joint" type="fixed">
-            <origin rpy="0 0 0" xyz="0 0.02 0" />
-            <parent link="head_camera_link" />
-            <child link="head_camera_rgb_frame" />
-        </joint>
-        <link name="head_camera_rgb_optical_frame" />
+            <origin rpy="0 0 0" xyz="0 0.02 0"/>
+            <parent link="head_camera_link"/>
+            <child link="head_camera_rgb_frame"/>
+        </joint>
+        <link name="head_camera_rgb_optical_frame"/>
         <joint name="head_camera_rgb_optical_joint" type="fixed">
-            <origin rpy="-1.57079632679 0 -1.57079632679" xyz="0 0 0" />
-            <parent link="head_camera_rgb_frame" />
-            <child link="head_camera_rgb_optical_frame" />
-        </joint>
-        <link name="head_camera_depth_frame" />
+            <origin rpy="-1.57079632679 0 -1.57079632679" xyz="0 0 0"/>
+            <parent link="head_camera_rgb_frame"/>
+            <child link="head_camera_rgb_optical_frame"/>
+        </joint>
+        <link name="head_camera_depth_frame"/>
         <joint name="head_camera_depth_joint" type="fixed">
-            <origin rpy="0 0 0" xyz="0 0.045 0" />
-            <parent link="head_camera_link" />
-            <child link="head_camera_depth_frame" />
-        </joint>
-        <link name="head_camera_depth_optical_frame" />
+            <origin rpy="0 0 0" xyz="0 0.045 0"/>
+            <parent link="head_camera_link"/>
+            <child link="head_camera_depth_frame"/>
+        </joint>
+        <link name="head_camera_depth_optical_frame"/>
         <joint name="head_camera_depth_optical_joint" type="fixed">
-            <origin rpy="-1.57079632679 0 -1.57079632679" xyz="0 0 0" />
-            <parent link="head_camera_depth_frame" />
-            <child link="head_camera_depth_optical_frame" />
+            <origin rpy="-1.57079632679 0 -1.57079632679" xyz="0 0 0"/>
+            <parent link="head_camera_depth_frame"/>
+            <child link="head_camera_depth_optical_frame"/>
         </joint>
         <link name="head_external_camera_mount">
             <inertial>
-                <origin rpy="0 0 0" xyz="0.00 -0.0025 0.013" />
-                <mass value="0.072" />
-                <inertia ixx="0.0061" ixy="-0.0" ixz="0.0002" iyy="0.0014" iyz="-0.0001" izz="0.0061" />
-            </inertial>
-            <visual>
-                <origin rpy="0 0 0" xyz="0 0 0" />
-                <geometry>
-                       <mesh filename="package://astro_description/meshes/head_external_camera_mount.stl" />
-                </geometry>
-                <material name="">
-                    <color rgba="0.20 0.20 0.20 1" />
-                </material>
-            </visual>
-            <collision>
-                <origin rpy="0 0 0" xyz="0 0 0" />
-                <geometry>
-                    <box size="0.099 0.020 0.023" />
+                <origin rpy="0 0 0" xyz="0.00 -0.0025 0.013"/>
+                <mass value="0.014"/>
+                <inertia ixx="13.42" ixy="-0.0" ixz="-0.107" iyy="2.998" iyz="0.000" izz="1.497"/>
+            </inertial>
+            <visual>
+                <origin rpy="0 0 0" xyz="0 0 0"/>
+                <geometry>
+                    <mesh filename="package://astro_description/meshes/head_external_camera_mount.stl"/>
+                </geometry>
+                <material name="">
+                    <color rgba="0.20 0.20 0.20 1"/>
+                </material>
+            </visual>
+            <collision>
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
Commit message: Add screen area to URDF
Gives a hook for gazebo video display plugin
Refactor material definitions

File: astro_description/urdf/head.xacro (robot description, xacro)
@@ -2,4 +2,10 @@
 <robot xmlns:xacro="http://www.ros.org/wiki/xacro" name="head">
     <xacro:include filename="$(find realsense2_description)/urdf/_d415.urdf.xacro"/>
+    <material name="ABS/IVR">
+        <color rgba="0.9 0.88 0.81 1"/>
+    </material>
+    <material name="ABS/BLK">
+        <color rgba="0.2 0.2 0.2 1"/>
+    </material>
     <xacro:macro name="head">
         <link name="head_pan_link">
@@ -54,7 +60,5 @@
                     <mesh filename="package://astro_description/meshes/xavier_mount.stl"/>
                 </geometry>
-                <material name="">
-                    <color rgba="0.2 0.2 0.2 1"/>
-                </material>
+                <material name="ABS/BLK"/>
             </visual>
             <collision>
@@ -110,7 +114,5 @@
                     <mesh filename="package://astro_description/meshes/display_mount.stl"/>
                 </geometry>
-                <material name="">
-                    <color rgba="0.2 0.2 0.16 1"/>
-                </material>
+                <material name="ABS/BLK"/>
             </visual>
             <collision>
@@ -137,7 +139,5 @@
                     <mesh filename="package://astro_description/meshes/head_display.stl"/>
                 </geometry>
-                <material name="">
-                    <color rgba="0.2 0.2 0.2 1"/>
-                </material>
+                <material name="ABS/BLK"/>
             </visual>
             <collision>
@@ -152,4 +152,23 @@
             <parent link="head_display_mount"/>
             <child link="head_display"/>
+        </joint>
+        <link name="head_display_screen">
+            <inertial>
+                <origin rpy="0 0 0" xyz="0 0 0"/>
+                <mass value="1.0"/>
+                <inertia ixx="0.0129" ixy="0.0002" ixz="0.0007" iyy="0.0095" iyz="-0.0" izz="0.0184"/>
+            </inertial>
+            <visual>
+                <origin rpy="0 0 0" xyz="0 0 0"/>
+                <geometry>
+                    <box size="0.2 0.12 0.001"/>
+                </geometry>
+                <material name="ABS/BLK"/>
+            </visual>
+        </link>
+        <joint name="head_display_screen_joint" type="fixed">
+            <origin rpy="0 0 0" xyz="0 0.007 0.0105"/>
+            <parent link="head_display"/>
+            <child link="head_display_screen"/>
         </joint>
         <link name="head_tilt_link">
@@ -233,7 +252,5 @@
                     <mesh filename="package://astro_description/meshes/head_external_camera_mount.stl"/>
                 </geometry>
-                <material name="">
-                    <color rgba="0.20 0.20 0.20 1"/>
-                </material>
+                <material name="ABS/BLK"/>
             </visual>
             <collision>
@@ -249,6 +266,6 @@
             <child link="head_external_camera_mount"/>
         </joint>
-        <xacro:arg name="use_nominal_extrinsics" default="True"/>
-        <sensor_d415 name="head_external_camera" parent="head_external_camera_mount" use_nominal_extrinsics="true">
+        <xacro:arg name="use_nominal_extrinsics" default="true"/>
+        <sensor_d415 name="head_external_camera" parent="head_external_camera_mount">
             <origin xyz="0.025 -0.025 0.003" rpy="0 0 0"/>
         </sensor_d415>
@@ -264,7 +281,5 @@
                     <mesh filename="package://astro_description/meshes/mic_mount.stl"/>
                 </geometry>
-                <material name="">
-                    <color rgba="0.20 0.20 0.20 1"/>
-                </material>
+                <material name="ABS/BLK"/>
             </visual>
             <collision>
@@ -291,7 +306,5 @@
                     <mesh filename="package://astro_description/meshes/mic.stl"/>
                 </geometry>
-                <material name="">
-                    <color rgba="0.20 0.20 0.20 1"/>
-                </material>
+                <material name="ABS/BLK"/>
             </visual>
             <collision>
@@ -318,7 +331,5 @@
                     <mesh filename="package://astro_description/meshes/mic_shell.stl"/>
                 </geometry>
-                <material name="">
-                    <color rgba="0.90 0.88 0.81 1"/>
-                </material>
+                <material name="ABS/IVR"/>
             </visual>
             <collision>
@@ -330,7 +341,7 @@
         </link>
         <joint name="mic_shell_joint" type="fixed">
-            <origin rpy="0 0 0" xyz="0.0 0.0 0.0" />
-            <parent link="head_mic_mount" />
-            <child link="mic_shell" />
+            <origin rpy="0 0 0" xyz="0.0 0.0 0.0"/>
+            <parent link="head_mic_mount"/>
+            <child link="mic_shell"/>
         </joint>
     </xacro:macro>
